Commit message: Modified the rviz visualization

File: gazebo_oru/euro_pallet/urdf/euro_pallet.xacro (robot description, xacro)
@@ -4,4 +4,5 @@
     <inertial>
       <mass value="2"/>
+      <!--  <mass value="2"/>  -->
       <inertia ixx="1" ixy="0" ixz="0" iyy="1" iyz="0" izz="1" />
       <origin/>

Commit message: Moved back to OrebroUniversity/navigation_oru-release master branch

File: gazebo_oru/euro_pallet/urdf/euro_pallet.xacro (robot description, xacro)
@@ -4,5 +4,4 @@
     <inertial>
       <mass value="2"/>
-      <!--  <mass value="2"/>  -->
       <inertia ixx="1" ixy="0" ixz="0" iyy="1" iyz="0" izz="1" />
       <origin/>
